Commit message: modify orbit_camera.urdf

File: orbit_pantilt/model/orbit_camera.urdf (robot description, URDF)
Before this commit: robot orbit_camera, 4 links, 3 joints
Links:
- removed link base
- removed link camera-link1
- removed link camera-link2
- removed link stick
- added link base_link; visual sphere radius=0.045
- added link camera_pan_link; visual sphere radius=0.035
- added link camera_tilt_link; visual cylinder length=0.01 radius=0.033; visual cylinder length=0.05 radius=0.01
- added link stick_link; visual cylinder length=0.22 radius=0.007
Joints:
- removed joint joint1
- added joint stick_joint: type fixed, parent base_link, child stick_link, origin xyz=0.01 0 0.05 rpy=0 0 0
- joint pan: child camera-link1 -> camera_pan_link; origin xyz=0 0 0.2 rpy=0 0 0 -> xyz=0 0 0.22 rpy=0 0 0; parent stick -> stick_link
- joint tilt: child camera-link2 -> camera_tilt_link; origin xyz=0 0 0.05 rpy=0 0 0 -> xyz=0 0 0.035 rpy=0 0 0; parent camera-link1 -> camera_pan_link

Commit message: enable orbit camera model to appear in the map with other robot

File: orbit_pantilt/model/orbit_camera.urdf (robot description, URDF)
Before this commit: robot orbit_camera, 4 links, 3 joints
Links:
- removed link base_link
- removed link camera_pan_link
- removed link camera_tilt_link
- removed link stick_link
- added link orbit_base_link; visual sphere radius=0.045
- added link orbit_camera_pan_link; visual sphere radius=0.035
- added link orbit_camera_tilt_link; visual cylinder length=0.01 radius=0.033; visual cylinder length=0.05 radius=0.01
- added link orbit_stick_link; visual cylinder length=0.22 radius=0.007
Joints:
- joint pan: child camera_pan_link -> orbit_camera_pan_link; parent stick_link -> orbit_stick_link
- joint stick_joint: child stick_link -> orbit_stick_link; parent base_link -> orbit_base_link
- joint tilt: child camera_tilt_link -> orbit_camera_tilt_link; parent camera_pan_link -> orbit_camera_pan_link

Commit message: fix orbit_camera.urdf for camera angle

File: orbit_pantilt/model/orbit_camera.urdf (robot description, URDF)
Before this commit: robot orbit_camera, 4 links, 3 joints
Joints:
- joint tilt: origin xyz=0 0 0.035 rpy=0 0 0 -> xyz=0 0 0.035 rpy=-1.57 0 -1.57
